Commit message: added 3d waypoints and paths, 2d sim is bugged atm

File: controller/scara_urdf/urdf/scara_urdf.urdf (robot description, URDF)
Before this commit: robot scara_urdf, 5 links, 4 joints
Links:
- link base_link: mass 2.4384 -> 2.4522
- link endR: mass 0.012412 -> 0.0124115438821334
Joints:
- joint jointz: limit lower=0 upper=0.08 effort=0 velocity=0 -> lower=1 upper=1 effort=0 velocity=0

Commit message: added axis marker, for some reason everything is red

File: controller/scara_urdf/urdf/scara_urdf.urdf (robot description, URDF)
Before this commit: robot scara_urdf, 5 links, 4 joints
Links:
- added link coordx, mass 0.0021586; collision mesh filename=package://scara_urdf/meshes/coordx.STL; visual mesh filename=package://scara_urdf/meshes/coordx.STL
- added link coordy, mass 0.0021586; collision mesh filename=package://scara_urdf/meshes/coordy.STL; visual mesh filename=package://scara_urdf/meshes/coordy.STL
- added link coordz, mass 0.0021586; collision mesh filename=package://scara_urdf/meshes/coordz.STL; visual mesh filename=package://scara_urdf/meshes/coordz.STL
- added link perimeter, mass 0; collision mesh filename=package://scara_urdf/meshes/perimeter.STL; visual mesh filename=package://scara_urdf/meshes/perimeter.STL
- link base_link: mass 2.4522 -> 2.43844795753921
- link endR: mass 0.0124115438821334 -> 0.0124115439277917
- link endZ: mass 0.0047788 -> 0.00477877779368
- link link1: mass 0.67597 -> 0.675965693614735
- link link2: mass 0.45238 -> 0.452384401379192
Joints:
- added joint coordx: type fixed, parent endR, child coordx, origin xyz=0 0 0 rpy=0 0 0, axis 0 0 0
- added joint coordy: type fixed, parent endR, child coordy, origin xyz=0 0 0 rpy=0 0 0, axis 0 0 0
- added joint coordz: type fixed, parent endR, child coordz, origin xyz=0 0 0 rpy=0 0 0, axis 0 0 0
- added joint perimeter: type fixed, parent base_link, child perimeter, origin xyz=0 0 0 rpy=0 0 0, axis 0 0 0
- joint jointz: origin xyz=0.18 0 0.12133 rpy=0 0 0 -> xyz=0.18 0 0.12109 rpy=0 0 0
